File: eda/drv10964/drv10964.kicad_sch (KiCad schematic)
At the start: 1 part

Commit message: exported drv10964 gerber files
Parts:
- added DRV1: ~, drv10964:drv10964, symbol drv10964:drv10964
- added J1, J2: Conn_01x05_Pin, Connector_PinHeader_2.54mm:PinHeader_1x05_P2.54mm_Vertical, symbol Connector:Conn_01x05_Pin
- added R1: 100k, Resistor_SMD:R_0603_1608Metric, symbol Device:R
- C1: value C -> 2.2uF; footprint (none) -> Capacitor_SMD:C_0603_1608Metric
Connections:
- net GND: now also DRV1.5 (GND), J2.5 (Pin_5)
- net VDD: now also DRV1.3 (VCC), J2.3 (Pin_3), R1.1
- new net CFG: DRV1.9 (CFG), J1.4 (Pin_4)
- new net FG: DRV1.1 (FG), J2.1 (Pin_1), R1.2
- new net FGS: DRV1.2 (FGS), J2.2 (Pin_2)
- new net FR: DRV1.8 (FR), J1.3 (Pin_3)
- new net PWM: DRV1.10 (PWM), J1.5 (Pin_5)
- new net U: DRV1.7 (U), J1.2 (Pin_2)
- new net V: DRV1.6 (V), J1.1 (Pin_1)
- new net W: DRV1.4 (W), J2.4 (Pin_4)
Other:
- moved on the sheet: C1
